Commit message: cleanup

File: triton_bringup/urdf/catamaran.urdf (robot description, URDF)
Before this commit: robot triton_bringup, 3 links, 2 joints
Links:
- link base_link: geometry collision mesh filename=file:///home/john/ros2_ws/src/Triton/triton_bringup/urdf/me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; visual mesh filename=file:///home/john/ros2_ws/src/Triton/triton_bringup/urdf/me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
- link imu_frame: geometry collision mesh filename=file:///home/john/ros2_ws/src/Triton/triton_bringup/urdf/me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; visual mesh filename=file:///home/john/ros2_ws/src/Triton/triton_bringup/urdf/me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
- link laser_frame: geometry collision mesh filename=file:///home/john/ros2_ws/src/Triton/triton_bringup/urdf/me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; visual mesh filename=file:///home/john/ros2_ws/src/Triton/triton_bringup/urdf/me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
